File: pteron_unibody_ec.kicad_pcb (KiCad board)
At the start: 2 copper layers, 255.8 x 141.9 mm, 99 parts, among them SW1 EC_SW, SW10 EC_SW, SW11 EC_SW, SW12 EC_SW, SW13 EC_SW, SW14 EC_SW, SW15 EC_SW, SW16 EC_SW, SW17 EC_SW, SW18 EC_SW, SW19 EC_SW, SW2 EC_SW, SW20 EC_SW, SW21 EC_SW, SW22 EC_SW, SW23 EC_SW, SW24 EC_SW, SW25 EC_SW, SW26 EC_SW, SW27 EC_SW, SW28 EC_SW, SW29 EC_SW, SW3 EC_SW, SW30 EC_SW, SW31 EC_SW, SW32 EC_SW, SW33 EC_SW, SW34 EC_SW, SW35 EC_SW, SW36 EC_SW, SW37 SW_Push, SW4 EC_SW, SW5 EC_SW, SW6 EC_SW, SW7 EC_SW, SW8 EC_SW, SW9 EC_SW, U2 74HC4051, U3 OPA350, U4 74HC4051, U5 ProMicro

Commit message: updated pcb with correct opamp schema and single source of mux sel
Parts:
- moved R11 11.5 mm to (196.6, 168.2)
- moved JP2 11.5 mm to (198.8, 168.1)
- moved R10 11.5 mm to (197.5, 171.4), turned to 180 degrees
- moved C3 1.24 mm to (202.8, 175.6)
Connections:
- U2 pad 10: /L_MUX_S1 -> /MUX_S1
- U2 pad 11: /L_MUX_S0 -> /MUX_S0
- U2 pad 9: /L_MUX_S2 -> /MUX_S2
- U3 pad 2: /DISCHARGE_PIN -> Net-(JP2-A)
- U3 pad 3: Net-(JP2-A) -> /DISCHARGE_PIN
- U4 pad 10: /R_MUX_S1 -> /MUX_S1
- U4 pad 11: /R_MUX_S0 -> /MUX_S0
- U4 pad 9: /R_MUX_S2 -> /MUX_S2
- U5 pad 10: /R_MUX_S2 -> unconnected-(U5-7/E6-Pad10)
- U5 pad 11: /R_MUX_S1 -> unconnected-(U5-8/B4-Pad11)
- U5 pad 12: /R_MUX_S0 -> /R_MUX_EN
- U5 pad 15: /L_MUX_S2 -> /MUX_S2
- U5 pad 16: /L_MUX_S1 -> /MUX_S1
- U5 pad 17: /L_MUX_S0 -> /MUX_S0
- U5 pad 9: /R_MUX_EN -> unconnected-(U5-6/D7-Pad9)
Routing:
- net /MUX_S0: track 0.00 -> 252.2 mm, vias 0 -> 1
- net /MUX_S1: track 0.00 -> 245.0 mm, vias 0 -> 1
- net /MUX_S2: track 0.00 -> 238.5 mm, vias 0 -> 1
- net /L_MUX_S0: track 120.2 -> 0.00 mm
- net /L_MUX_S1: track 116.1 -> 0.00 mm
- net /L_MUX_S2: track 113.9 -> 0.00 mm
- net /R_MUX_S2: track 111.8 -> 0.00 mm
- net /R_MUX_S1: track 111.7 -> 0.00 mm
- net /R_MUX_S0: track 111.5 -> 0.00 mm
- net /R_MUX_EN: track 111.6 -> 104.0 mm
- net Net-(JP2-A): track 10.1 -> 11.7 mm
- net /COL7: track 168.0 -> 166.6 mm
- net /DISCHARGE_PIN: track 231.0 -> 232.1 mm
- net /ADC: track 58.7 -> 59.5 mm
- net GND: vias 259 -> 268

Commit message: updated trace with fillet
Parts:
- R1, R2, R3: moved to F.Cu
- moved R4 3.35 mm to (175.0, 186.5), turned to -150 degrees
- moved R3 1.69 mm to (205.8, 124.7)
- moved C5 0.62 mm to (201.8, 161.5)
- moved SW9 0.54 mm to (154.8, 138.0)
- moved SW14 0.54 mm to (148.3, 155.8)
- moved R1 0.54 mm to (204.1, 114.5)
- moved H37 0.54 mm to (203.6, 220.0)
- moved SW26 0.54 mm to (274.4, 143.7)
- moved U4 0.54 mm to (283.1, 167.3)
- moved H34 0.54 mm to (255.4, 146.9)
- moved H6 0.54 mm to (168.7, 155.3)
- moved SW12 0.54 mm to (112.9, 141.9)
- moved SW30 0.54 mm to (231.0, 200.2)
- moved SW31 0.54 mm to (307.7, 113.3)
- moved SW24 0.54 mm to (261.5, 108.0)
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Routing:
- net Net-(R3-Pad2): track 301.3 -> 316.7 mm, vias 12 -> 11
- net Net-(R1-Pad2): track 257.9 -> 272.4 mm, vias 10 -> 11
- net /COL1: track 206.1 -> 216.6 mm
- net Net-(R2-Pad2): track 282.3 -> 292.6 mm, vias 12 -> 11
- net Net-(R4-Pad2): track 134.0 -> 143.5 mm
- net /COL2: track 169.3 -> 178.2 mm
- net /COL7: track 166.6 -> 157.9 mm
- net /ROW3: track 83.4 -> 92.0 mm
- net /MUX_S0: track 252.2 -> 260.6 mm
- net /MUX_S1: track 245.0 -> 253.1 mm
- net /MUX_S2: track 238.5 -> 246.3 mm
- net /COL9: track 219.6 -> 225.5 mm
- net /COL5: track 110.9 -> 115.7 mm
- net /COL4: track 114.3 -> 118.6 mm
- net /COL8: track 192.7 -> 196.9 mm
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
Commit message: updated traces and 3d footprints
Parts:
- added J1: Conn_01x05, pteron_unibody_ec:nice_view, F.Cu at (201.6, 130.5)
- R1, R2, R3: moved to B.Cu
- moved R4 70.8 mm to (203.2, 121.7), turned to 180 degrees
- moved R3 5.67 mm to (203.2, 119.6)
- moved R10 1.86 mm to (195.9, 171.2)
- moved R18 1.86 mm to (298.0, 162.8)
- moved H2 1.86 mm to (162.7, 111.5)
- moved JP2 1.86 mm to (197.1, 167.9)
- moved H21 1.86 mm to (275.9, 152.9)
- moved R12 1.86 mm to (285.0, 158.7)
- moved R8 1.86 mm to (101.1, 161.7)
- moved H25 1.86 mm to (313.2, 141.0)
- moved U4 1.86 mm to (281.3, 167.5)
- moved SW12 1.86 mm to (111.1, 142.2)
- moved SW2 1.86 mm to (124.1, 106.5)
- moved H34 1.86 mm to (253.5, 147.2)
- moved H20 1.86 mm to (222.0, 208.7)
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Connections:
- U5 pad 1: /ROW0 -> unconnected-(U5-TX0/D3-Pad1)
- U5 pad 10: unconnected-(U5-7/E6-Pad10) -> /ROW2
- U5 pad 11: unconnected-(U5-8/B4-Pad11) -> /ROW3
- U5 pad 2: /ROW1 -> unconnected-(U5-RX1/D2-Pad2)
- U5 pad 5: /ROW2 -> /MOSI
- U5 pad 6: /ROW3 -> /SCK
- U5 pad 7: unconnected-(U5-4/D4-Pad7) -> /CS
- U5 pad 8: unconnected-(U5-5/C6-Pad8) -> /ROW0
- U5 pad 9: unconnected-(U5-6/D7-Pad9) -> /ROW1
Routing:
- net Net-(R4-Pad2): track 143.5 -> 231.7 mm, vias 6 -> 8
- net /ROW3: track 92.0 -> 22.3 mm, vias 1 -> 0
- net /CS: track 0.00 -> 33.9 mm
- net /MOSI: track 0.00 -> 31.0 mm
- net /SCK: track 0.00 -> 28.6 mm
- net /ROW2: track 4.36 -> 22.0 mm
- net Net-(R2-Pad2): track 292.6 -> 309.4 mm, vias 11 -> 10
- net +3.3V: track 257.3 -> 272.5 mm
- net /ROW1: track 6.00 -> 20.7 mm
- net Net-(R3-Pad2): track 316.7 -> 331.2 mm, vias 11 -> 12
- net /ROW0: track 6.00 -> 20.5 mm
- net Net-(R1-Pad2): track 272.4 -> 282.8 mm, vias 11 -> 10
- net /ADC: track 59.0 -> 53.9 mm
- net /COL7: track 157.9 -> 163.0 mm
- net /MUX_S1: track 253.1 -> 251.9 mm, vias 1 -> 3
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