File: pteron_unibody_ec.kicad_sch (KiCad schematic)
At the start: 62 parts, among them SW1 EC_SW, SW10 EC_SW, SW11 EC_SW, SW12 EC_SW, SW13 EC_SW, SW14 EC_SW, SW15 EC_SW, SW16 EC_SW, SW17 EC_SW, SW18 EC_SW, SW19 EC_SW, SW2 EC_SW, SW20 EC_SW, SW21 EC_SW, SW22 EC_SW, SW23 EC_SW, SW24 EC_SW, SW25 EC_SW, SW26 EC_SW, SW27 EC_SW, SW28 EC_SW, SW29 EC_SW, SW3 EC_SW, SW30 EC_SW, SW31 EC_SW, SW32 EC_SW, SW33 EC_SW, SW34 EC_SW, SW35 EC_SW, SW36 EC_SW, SW37 SW_Push, SW4 EC_SW, SW5 EC_SW, SW6 EC_SW, SW7 EC_SW, SW8 EC_SW, SW9 EC_SW, U2 74HC4051, U3 OPA350, U4 74HC4051, U5 ProMicro

Commit message: updated pcb with correct opamp schema and single source of mux sel
Connections:
- net DISCHARGE_PIN: now also U3.3 (IN+); no longer U3.2 (IN-)
- net R_MUX_EN: now also U5.12 (9/B5); no longer U5.9 (6/D7)
- net at JP2.1 (A), R10.1, R11.1: now also U3.2 (IN-); no longer U3.3 (IN+)
- net L_MUX_S0 renamed MUX_S0
- net MUX_S0: now also U4.11 (S0)
- net L_MUX_S1 renamed MUX_S1
- net MUX_S1: now also U4.10 (S1)
- net L_MUX_S2 renamed MUX_S2
- net MUX_S2: now also U4.9 (S2)
- removed net R_MUX_S0: U4.11 (S0), U5.12 (9/B5)
- net R_MUX_S1: no longer names the net of U5.11 (8/B4)
- net R_MUX_S1: no longer U4.10 (S1)
- net R_MUX_S2: no longer names the net of U5.10 (7/E6)
- net R_MUX_S2: no longer U4.9 (S2)
Other:
- moved on the sheet: C3

Commit message: updated traces and 3d footprints
Parts:
- added J1: Conn_01x05, pteron_unibody_ec:nice_view, symbol Connector_Generic:Conn_01x05
Connections:
- net +3.3V: now also J1.3 (Pin_3)
- net GND: now also J1.4 (Pin_4)
- net ROW0: now also U5.8 (5/C6); no longer U5.1 (TX0/D3)
- net ROW1: now also U5.9 (6/D7); no longer U5.2 (RX1/D2)
- net ROW2: now also U5.10 (7/E6); no longer U5.5 (2/D1/SDA)
- net ROW3: now also U5.11 (8/B4); no longer U5.6 (3/D0/SCL)
- net CS: now reaches U5.7 (4/D4)
- net CS: now also J1.5 (Pin_5)
- new net MOSI: J1.1 (Pin_1), U5.5 (2/D1/SDA)
- new net SCK: J1.2 (Pin_2), U5.6 (3/D0/SCL)
- no-connect marks 5 -> 3
Changed lines of the file:
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@@
   (no_connect (at 68.707 179.07))
   (no_connect (at 68.707 181.61))
-  (no_connect (at 33.147 181.61))
   (no_connect (at 68.707 166.37))
-  (no_connect (at 33.147 184.15))
   (wire (pts (xy 229.87 52.07) (xy 229.87 59.69))
     (stroke (width 0) (type default))
@@
     (stroke (width 0) (type default))
   )
-  (wire (pts (xy 25.019 168.91) (xy 33.147 168.91))
+  (wire (pts (xy 25.019 186.69) (xy 33.147 186.69))
     (stroke (width 0) (type default))
   )
@@
     (stroke (width 0) (type default))
   )
-  (wire (pts (xy 24.765 166.37) (xy 33.147 166.37))
+  (wire (pts (xy 24.765 184.15) (xy 33.147 184.15))
     (stroke (width 0) (type default))
   )
@@
     (stroke (width 0) (type default))
   )
-  (wire (pts (xy 24.511 176.53) (xy 33.147 176.53))
+  (wire (pts (xy 24.511 189.23) (xy 33.147 189.23))
     (stroke (width 0) (type default))
   )
@@
     (stroke (width 0) (type default))
   )
-  (wire (pts (xy 24.511 179.07) (xy 33.147 179.07))
+  (wire (pts (xy 24.511 191.77) (xy 33.147 191.77))
     (stroke (width 0) (type default))
   )
@@
     (effects (font (size 1.27 1.27)) (justify right bottom))
   )
+  (label "SCK" (at 33.147 179.07 180) (fields_autoplaced)
+    (effects (font (size 1.27 1.27)) (justify right bottom))
+  )
   (label "COL5" (at 269.113 131.318 0) (fields_autoplaced)
     (effects (font (size 1.27 1.27)) (justify left bottom))
@@
     (effects (font (size 1.27 1.27)) (justify right bottom))
   )
+  (label "MOSI" (at 33.147 176.53 180) (fields_autoplaced)
+    (effects (font (size 1.27 1.27)) (justify right bottom))
+  )
   (label "ADC" (at 68.707 176.53 0) (fields_autoplaced)
     (effects (font (size 1.27 1.27)) (justify left bottom))
@@
     (effects (font (size 1.27 1.27)) (justify right bottom))
   )
-  (label "ROW2" (at 24.511 176.53 180) (fields_autoplaced)
+  (label "ROW2" (at 24.511 189.23 180) (fields_autoplaced)
     (effects (font (size 1.27 1.27)) (justify right bottom))
   )
@@
     (effects (font (size 1.27 1.27)) (justify left bottom))
   )
-  (label "ROW0" (at 24.765 166.37 180) (fields_autoplaced)
+  (label "ROW0" (at 24.765 184.15 180) (fields_autoplaced)
     (effects (font (size 1.27 1.27)) (justify right bottom))
   )
@@
     (effects (font (size 1.27 1.27)) (justify right bottom))
   )
-  (label "ROW1" (at 25.019 168.91 180) (fields_autoplaced)
+  (label "SCK" (at 148.59 168.656 180) (fields_autoplaced)
+    (effects (font (size 1.27 1.27)) (justify right bottom))
+  )
+  (label "ROW1" (at 25.019 186.69 180) (fields_autoplaced)
     (effects (font (size 1.27 1.27)) (justify right bottom))
   )
@@
     (effects (font (size 1.27 1.27)) (justify right bottom))
   )
+  (label "MOSI" (at 148.59 166.116 180) (fields_autoplaced)
+    (effects (font (size 1.27 1.27)) (justify right bottom))
+  )
   (label "MUX_S0" (at 214.503 123.698 180) (fields_autoplaced)
     (effects (font (size 1.27 1.27)) (justify right bottom))
@@
     (effects (font (size 1.27 1.27)) (justify left bottom))
   )
+  (label "CS" (at 33.147 181.61 180) (fields_autoplaced)
+    (effects (font (size 1.27 1.27)) (justify right bottom))
+  )
   (label "COL2" (at 83.185 120.142 0) (fields_autoplaced)
     (effects (font (size 1.27 1.27)) (justify left bottom))
@@
     (effects (font (size 1.27 1.27)) (justify right bottom))
   )
-  (label "ROW3" (at 24.511 179.07 180) (fields_autoplaced)
+  (label "ROW3" (at 24.511 191.77 180) (fields_autoplaced)
+    (effects (font (size 1.27 1.27)) (justify right bottom))
+  )
+  (label "CS" (at 148.59 176.276 180) (fields_autoplaced)
     (effects (font (size 1.27 1.27)) (justify right bottom))
   )
@@
   )
   (symbol (lib_id "power:GND") (at 33.147 173.99 270) (unit 1)
-    (in_bom yes) (on_board yes) (dnp no) (fields_autoplaced)
+    (in_bom yes) (on_board yes) (dnp no)
     (property "Reference" "#PWR027" (at 26.797 173.99 0)
       (effects (font (size 1.27 1.27)) hide)
@@
     )
   )
+  (symbol (lib_id "Connector_Generic:Conn_01x05") (at 153.67 171.196 0) (unit 1)
+    (in_bom yes) (on_board yes) (dnp no) (fields_autoplaced)
+    (property "Reference" "J1" (at 156.21 169.926 0)
+      (effects (font (size 1.27 1.27)) (justify left))
+    )
+    (property "Value" "Conn_01x05" (at 156.21 172.466 0)
+      (effects (font (size 1.27 1.27)) (justify left))
+    )
+    (property "Footprint" "pteron_unibody_ec:nice_view" (at 153.67 171.196 0)
+      (effects (font (size 1.27 1.27)) hide)
+    )
+    (property "Datasheet" "~" (at 153.67 171.196 0)
+      (effects (font (size 1.27 1.27)) hide)
+    )
+    (pin "1")
+    (pin "2")
+    (pin "3")
+    (pin "4")
+    (pin "5")
+    (instances
+      (project "pteron_unibody_ec"
+        (path "/c4f0c9d7-85ec-4361-a16b-3fe1005ec647"
+          (reference "J1") (unit 1)
+        )
+      )
+    )
+  )
   (symbol (lib_id "pteron_unibody:EC_SW") (at 36.83 67.31 0) (unit 1)
     (in_bom yes) (on_board yes) (dnp no) (fields_autoplaced)
@@
     )
   )
+  (symbol (lib_id "power:+3.3V") (at 148.59 171.196 90) (unit 1)
+    (in_bom yes) (on_board yes) (dnp no) (fields_autoplaced)
+    (property "Reference" "#PWR024" (at 152.4 171.196 0)
+      (effects (font (size 1.27 1.27)) hide)
+    )
+    (property "Value" "+3.3V" (at 145.034 171.196 90)
+      (effects (font (size 1.27 1.27)) (justify left))
+    )
+    (property "Footprint" "" (at 148.59 171.196 0)
+      (effects (font (size 1.27 1.27)) hide)
+    )
+    (property "Datasheet" "" (at 148.59 171.196 0)
+      (effects (font (size 1.27 1.27)) hide)
+    )
+    (pin "1")
+    (instances
+      (project "pteron_unibody_ec"
+        (path "/c4f0c9d7-85ec-4361-a16b-3fe1005ec647"
+          (reference "#PWR024") (unit 1)
+        )
+      )
+    )
+  )
   (symbol (lib_id "pteron_unibody:EC_SW") (at 36.83 35.56 0) (unit 1)
     (in_bom yes) (on_board yes) (dnp no) (fields_autoplaced)
@@
     )
   )
+  (symbol (lib_id "power:GND") (at 148.59 173.736 270) (unit 1)
+    (in_bom yes) (on_board yes) (dnp no) (fields_autoplaced)
+    (property "Reference" "#PWR028" (at 142.24 173.736 0)
+      (effects (font (size 1.27 1.27)) hide)
+    )
+    (property "Value" "GND" (at 144.653 173.736 90)
+      (effects (font (size 1.27 1.27)) (justify right))
+    )
+    (property "Footprint" "" (at 148.59 173.736 0)
+      (effects (font (size 1.27 1.27)) hide)
+    )
+    (property "Datasheet" "" (at 148.59 173.736 0)
+      (effects (font (size 1.27 1.27)) hide)
+    )
+    (pin "1")
+    (instances
+      (project "pteron_unibody_ec"
+        (path "/c4f0c9d7-85ec-4361-a16b-3fe1005ec647"
+          (reference "#PWR028") (unit 1)
+        )
+      )
+    )
+  )
   (symbol (lib_id "pteron_unibody:EC_SW") (at 96.52 52.07 0) (unit 1)
     (in_bom yes) (on_board yes) (dnp no) (fields_autoplaced)
@@
     )
   )
-  (sheet (at 122.555 169.291) (size 18.923 5.588) (fields_autoplaced)
+  (sheet (at 98.679 162.306) (size 18.923 5.588) (fields_autoplaced)
     (stroke (width 0.1524) (type solid))
     (fill (color 0 0 0 0.0000))
-    (property "Sheetname" "Mounting_holes" (at 122.555 168.5794 0)
+    (property "Sheetname" "Mounting_holes" (at 98.679 161.5944 0)
       (effects (font (size 1.27 1.27)) (justify left bottom))
     )
-    (property "Sheetfile" "mounting.kicad_sch" (at 122.555 175.4636 0)
+    (property "Sheetfile" "mounting.kicad_sch" (at 98.679 168.4786 0)
       (effects (font (size 1.27 1.27)) (justify left top))
     )

Commit message: final version
Parts:
- added L1: ART, personal-logo:peacock-large, symbol Mechanical:MountingHole
- added L2: ART, personal-logo:peacock-medium, symbol Mechanical:MountingHole
- J1: value Conn_01x05 -> Nice!view display
Other:
- moved on the sheet: J1
Changed lines of the file:
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@@
+    (fill (type none))
+  )
+  (rectangle (start 146.939 160.02) (end 169.799 178.689)
+    (stroke (width 0) (type default))
     (fill (type none))
   )
@@
     (fill (type none))
   )
+  (rectangle (start 123.19 159.766) (end 142.494 180.594)
+    (stroke (width 0) (type default))
+    (fill (type none))
+  )
   (rectangle (start 150.495 20.32) (end 283.845 99.695)
     (stroke (width 0) (type default))
@@
     (effects (font (size 1.27 1.27)) (justify right bottom))
   )
-  (label "SCK" (at 148.59 168.656 180) (fields_autoplaced)
+  (label "SCK" (at 132.334 167.132 180) (fields_autoplaced)
     (effects (font (size 1.27 1.27)) (justify right bottom))
   )
@@
     (effects (font (size 1.27 1.27)) (justify right bottom))
   )
-  (label "MOSI" (at 148.59 166.116 180) (fields_autoplaced)
+  (label "MOSI" (at 132.334 164.592 180) (fields_autoplaced)
     (effects (font (size 1.27 1.27)) (justify right bottom))
   )
@@
     (effects (font (size 1.27 1.27)) (justify right bottom))
   )
-  (label "CS" (at 148.59 176.276 180) (fields_autoplaced)
+  (label "CS" (at 132.334 174.752 180) (fields_autoplaced)
     (effects (font (size 1.27 1.27)) (justify right bottom))
   )
@@
     )
   )
-  (symbol (lib_id "Connector_Generic:Conn_01x05") (at 153.67 171.196 0) (unit 1)
-    (in_bom yes) (on_board yes) (dnp no) (fields_autoplaced)
-    (property "Reference" "J1" (at 156.21 169.926 0)
-      (effects (font (size 1.27 1.27)) (justify left))
-    )
-    (property "Value" "Conn_01x05" (at 156.21 172.466 0)
-      (effects (font (size 1.27 1.27)) (justify left))
-    )
-    (property "Footprint" "pteron_unibody_ec:nice_view" (at 153.67 171.196 0)
-      (effects (font (size 1.27 1.27)) hide)
-    )
-    (property "Datasheet" "~" (at 153.67 171.196 0)
+  (symbol (lib_id "Connector_Generic:Conn_01x05") (at 137.414 169.672 0) (unit 1)
+    (in_bom yes) (on_board yes) (dnp no)
+    (property "Reference" "J1" (at 139.954 168.402 0)
+      (effects (font (size 1.27 1.27)) (justify left))
+    )
+    (property "Value" "Nice!view display" (at 125.349 177.927 0)
+      (effects (font (size 1.27 1.27)) (justify left))
+    )
+    (property "Footprint" "pteron_unibody_ec:nice_view" (at 137.414 169.672 0)
+      (effects (font (size 1.27 1.27)) hide)
+    )
+    (property "Datasheet" "~" (at 137.414 169.672 0)
       (effects (font (size 1.27 1.27)) hide)
     )
@@
         (path "/c4f0c9d7-85ec-4361-a16b-3fe1005ec647"
           (reference "SW23") (unit 1)
+        )
+      )
+    )
+  )
+  (symbol (lib_id "Mechanical:MountingHole") (at 157.861 173.736 0) (unit 1)
+    (in_bom yes) (on_board yes) (dnp no) (fields_autoplaced)
+    (property "Reference" "L2" (at 160.528 172.466 0)
+      (effects (font (size 1.27 1.27)) (justify left))
+    )
+    (property "Value" "ART" (at 160.528 175.006 0)
+      (effects (font (size 1.27 1.27)) (justify left))
+    )
+    (property "Footprint" "personal-logo:peacock-medium" (at 157.861 173.736 0)
+      (effects (font (size 1.27 1.27)) hide)
+    )
+    (property "Datasheet" "~" (at 157.861 173.736 0)
+      (effects (font (size 1.27 1.27)) hide)
+    )
+    (instances
+      (project "pteron_unibody_ec"
+        (path "/c4f0c9d7-85ec-4361-a16b-3fe1005ec647"
+          (reference "L2") (unit 1)
         )
       )
@@
     )
   )
+  (symbol (lib_id "Mechanical:MountingHole") (at 152.273 166.751 0) (unit 1)
+    (in_bom yes) (on_board yes) (dnp no) (fields_autoplaced)
+    (property "Reference" "L1" (at 154.94 165.481 0)
+      (effects (font (size 1.27 1.27)) (justify left))
+    )
+    (property "Value" "ART" (at 154.94 168.021 0)
+      (effects (font (size 1.27 1.27)) (justify left))
+    )
+    (property "Footprint" "personal-logo:peacock-large" (at 152.273 166.751 0)
+      (effects (font (size 1.27 1.27)) hide)
+    )
+    (property "Datasheet" "~" (at 152.273 166.751 0)
+      (effects (font (size 1.27 1.27)) hide)
+    )
+    (instances
+      (project "pteron_unibody_ec"
+        (path "/c4f0c9d7-85ec-4361-a16b-3fe1005ec647"
+          (reference "L1") (unit 1)
+        )
+      )
+    )
+  )
   (symbol (lib_id "power:+3.3V") (at 68.707 173.99 270) (unit 1)
     (in_bom yes) (on_board yes) (dnp no) (fields_autoplaced)
@@
     )
   )
-  (symbol (lib_id "power:+3.3V") (at 148.59 171.196 90) (unit 1)
-    (in_bom yes) (on_board yes) (dnp no) (fields_autoplaced)
-    (property "Reference" "#PWR024" (at 152.4 171.196 0)
-      (effects (font (size 1.27 1.27)) hide)
-    )
-    (property "Value" "+3.3V" (at 145.034 171.196 90)
-      (effects (font (size 1.27 1.27)) (justify left))
-    )
-    (property "Footprint" "" (at 148.59 171.196 0)
-      (effects (font (size 1.27 1.27)) hide)
-    )
-    (property "Datasheet" "" (at 148.59 171.196 0)
+  (symbol (lib_id "power:+3.3V") (at 132.334 169.672 90) (unit 1)
+    (in_bom yes) (on_board yes) (dnp no) (fields_autoplaced)
+    (property "Reference" "#PWR024" (at 136.144 169.672 0)
+      (effects (font (size 1.27 1.27)) hide)
+    )
+    (property "Value" "+3.3V" (at 128.778 169.672 90)
+      (effects (font (size 1.27 1.27)) (justify left))
+    )
+    (property "Footprint" "" (at 132.334 169.672 0)
+      (effects (font (size 1.27 1.27)) hide)
+    )
+    (property "Datasheet" "" (at 132.334 169.672 0)
       (effects (font (size 1.27 1.27)) hide)
     )
@@
     )
   )
-  (symbol (lib_id "power:GND") (at 148.59 173.736 270) (unit 1)
-    (in_bom yes) (on_board yes) (dnp no) (fields_autoplaced)
-    (property "Reference" "#PWR028" (at 142.24 173.736 0)
-      (effects (font (size 1.27 1.27)) hide)
-    )
-    (property "Value" "GND" (at 144.653 173.736 90)
+  (symbol (lib_id "power:GND") (at 132.334 172.212 270) (unit 1)
+    (in_bom yes) (on_board yes) (dnp no) (fields_autoplaced)
+    (property "Reference" "#PWR028" (at 125.984 172.212 0)
+      (effects (font (size 1.27 1.27)) hide)
+    )
+    (property "Value" "GND" (at 128.397 172.212 90)
       (effects (font (size 1.27 1.27)) (justify right))
     )
-    (property "Footprint" "" (at 148.59 173.736 0)
-      (effects (font (size 1.27 1.27)) hide)
-    )
-    (property "Datasheet" "" (at 148.59 173.736 0)
-      (effects (font (size 1.27 1.27)) hide)
-    )
+    (property "Footprint" "" (at 132.334 172.212 0)
+      (effects (font (size 1.27 1.27)) hide)
+    )
+    (property "Datasheet" "" (at 132.334 172.212 0)
+      (effects (font (size 1.27 1.27)) hide)
+    )
